Commit message: flipped lidar 180 and slowed down nav2

File: urdf/ursula.urdf.xacro (robot description, xacro)
@@ -198,5 +198,5 @@
   <xacro:ursula_wheels parent="chassis_link"/>
   <xacro:slamtec_rplidar_a3 parent="chassis_link">
-    <origin xyz="${chassis_length / 2.0 - 0.2419} 0 ${0.4485 - chassis_center_z}" rpy="0 0 0"/>
+    <origin xyz="${chassis_length / 2.0 - 0.2419} 0 ${0.4485 - chassis_center_z}" rpy="0 0 3.14159"/>
   </xacro:slamtec_rplidar_a3>
   <xacro:luxonis_oak_d parent="chassis_link">

Commit message: robot orientation

File: urdf/ursula.urdf.xacro (robot description, xacro)
@@ -194,9 +194,9 @@
     <parent link="base_link"/>
     <child  link="chassis_link"/>
-    <origin xyz="0 0 ${chassis_center_z}" rpy="0 0 3.14159"/>
+    <origin xyz="0 0 ${chassis_center_z}" rpy="0 0 0"/>
   </joint>
   <xacro:ursula_wheels parent="chassis_link"/>
   <xacro:slamtec_rplidar_a3 parent="chassis_link">
-    <origin xyz="${chassis_length / 2.0 - 0.2419} 0 ${0.4485 - chassis_center_z}" rpy="0 0 0"/>
+    <origin xyz="${chassis_length / 2.0 - 0.2419} 0 ${0.4485 - chassis_center_z}" rpy="0 0 3.14159"/>
   </xacro:slamtec_rplidar_a3>
   <xacro:luxonis_oak_d parent="chassis_link">
